File: arduino-nano-drone/radio-receiver/arduino-nano-radio-receiver.kicad_pcb (KiCad board)
At the start: 2 copper layers, 38 x 63.3 mm, 11 parts

Commit message: Reviewed schematics and boards
Other:
- board text added: "Kondensator na in/out przetwornicy"
- board text added: "Kondensator na wejściu RF"
- board text added: "Spokojnie zrób grubsze ścieżki 12v, masz dużo miejsca"
Changed lines of the file:
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@@
+    (effects (font (size 1 1) (thickness 0.15)) (justify left bottom))
+  )
+  (gr_text "Kondensator na in/out przetwornicy " (at 107.925 71.2) (layer "User.8")
+    (effects (font (size 1 1) (thickness 0.15)) (justify left bottom))
+  )
+  (gr_text "Kondensator na wejściu RF" (at 112.525 46.675) (layer "User.8")
+    (effects (font (size 1 1) (thickness 0.15)) (justify left bottom))
+  )
+  (gr_text "Spokojnie zrób grubsze ścieżki 12v, masz dużo miejsca" (at 94.225 84.275) (layer "User.8")
     (effects (font (size 1 1) (thickness 0.15)) (justify left bottom))
   )

Commit message: project 8 / arduino nano drone / improved schematics, pcb after review
Parts:
- added C1: 10u, Capacitor_THT:CP_Radial_D4.0mm_P1.50mm, F.Cu at (108.6, 79.6)
- added C2: 10u, Capacitor_THT:CP_Radial_D4.0mm_P1.50mm, F.Cu at (114.0, 41.6)
- moved U2 4.40 mm to (113.3, 45.8)
- moved U1 1.52 mm to (105.5, 75.4)
- moved BT1 0.25 mm to (104.6, 84.0)
- moved J1 0.25 mm to (110.8, 84.0)
- renumbered ARDUINO to A1, PPM to J1, AMS1117 to U1, NRF24 to U2
Connections:
- A1 pad 11: unconnected-(A1-D8-Pad11) -> /IRQ
- U2 pad 8: unconnected-(U2-IRQ-Pad8) -> /IRQ
Routing:
- net +3.3V: track 32.4 -> 44.4 mm
- net /IRQ: track 0.00 -> 11.4 mm
- net Net-(A1-D2): track 17.9 -> 22.2 mm
- net /CE: track 19.1 -> 16.2 mm
- net /CSN: track 16.1 -> 14.1 mm
- net /MISO: track 9.93 -> 8.01 mm
- net +12V: track 35.7 -> 36.7 mm
- net /SCK: track 27.7 -> 26.8 mm
- net /MOSI: track 12.5 -> 11.5 mm
- net GND: track 0.41 -> 0.00 mm, vias 23 -> 22
Other:
- board text removed: "Kondensator na in/out przetwornicy"
- board text removed: "Kondensator na wejściu RF"
- board text removed: "Spokojnie zrób grubsze ścieżki 12v, masz dużo miejsca"
