File: arduino-nano-drone/radio-transmitter/arduino-nano-radio-transmitter.kicad_pcb (KiCad board)
At the start: 2 copper layers, 41.1 x 68.8 mm, 14 parts, among them U3 NRF24L01_Breakout

Commit message: Reviewed schematics and boards
Other:
- board text added: "A z czego będzie te 12V? upewnij się, że nie ma szans na skok do np 12.5-14"
- board text added: "Jak jest miejsce, to spokojnie rób szersze ścieżki na zasilanie. W razie czego puści więcej prądu, nie będzie brzydkich spadków itp."
- board text added: "Poddtrzymuję, dodatkowy kondek tutaj nie zaszkodzi"
- board text added: "Te przelotki tu nic nie wniosą jbc. Ścieżki są i tak za daleko od siebie"
Changed lines of the file:
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@@
     (effects (font (size 1 1) (thickness 0.15)) (justify left bottom))
+  )
+  (gr_text "Poddtrzymuję, dodatkowy kondek tutaj nie zaszkodzi" (at 107.425 68.35) (layer "User.8")
+    (effects (font (size 1 1) (thickness 0.15)) (justify left bottom))
+  )
+  (gr_text "Te przelotki tu nic nie wniosą jbc. Ścieżki są i tak za daleko od siebie" (at 93.775 51.6) (layer "User.8")
+    (effects (font (size 1 1) (thickness 0.15)) (justify left bottom))
+  )
+  (gr_text "A z czego będzie te 12V? upewnij się, że nie ma szans na skok do np 12.5-14" (at 107.475 45.4) (layer "User.8")
+    (effects (font (size 1 1) (thickness 0.15)) (justify left bottom))
+  )
+  (gr_text "Jak jest miejsce, to spokojnie rób szersze ścieżki na zasilanie. W razie czego puści więcej prądu, nie będzie brzydkich spadków itp." (at 102 60.475) (layer "User.8")
+    (effects (font (size 1.5 1.5) (thickness 0.3) bold) (justify left bottom))
   )
   (via (at 92.5 66.3) (size 0.8) (drill 0.4) (layers "F.Cu" "B.Cu") (net 0))
@@
         (xy 117 104.1)
         (xy 69 104.4)
-        (xy 69 31.4)
-        (xy 69 31.4)
-        (xy 69 31.4)
       )
     )

Commit message: project 8 / arduino nano drone / improved schematics, pcb after review
Parts:
- added C2: 10u, Capacitor_THT:CP_Radial_D4.0mm_P1.50mm, F.Cu at (107.0, 53.9)
- added C3: 100n, Capacitor_THT:C_Disc_D3.0mm_W1.6mm_P2.50mm, F.Cu at (106.7, 50.5)
- moved U2 1.87 mm to (96.3, 60.2)
- moved C1 1.72 mm to (107.0, 59.9)
- moved J2 1.44 mm to (99.7, 44.9)
- moved BT1 1.44 mm to (107.8, 44.9)
- moved J1 1.44 mm to (96.0, 44.9)
- moved J3 1.44 mm to (103.2, 44.9)
- moved U3 0.90 mm to (108.0, 63.9)
- renumbered POT to J1, 5V to J2, GND to J3, AMS to U2
Connections:
- A1 pad 11: unconnected-(A1-D8-Pad11) -> /IRQ
- U3 pad 8: unconnected-(U3-IRQ-Pad8) -> /IRQ
Routing:
- net /IRQ: track 0.00 -> 27.4 mm
- net +3.3V: track 16.2 -> 22.9 mm
- net +12V: track 73.1 -> 77.5 mm
- net Net-(A1-A0): track 14.3 -> 16.6 mm
- net Net-(A1-A1): track 14.6 -> 16.3 mm
- net Net-(A1-A2): track 14.6 -> 16.2 mm
- net Net-(A1-A3): track 14.6 -> 16.2 mm
- net /SCK: track 20.5 -> 21.7 mm
- net Net-(A1-+5V): track 38.1 -> 39.0 mm
- net /MISO: track 34.9 -> 34.1 mm
- net GND: vias 34 -> 32
Other:
- board text removed: "A z czego będzie te 12V? upewnij się, że nie ma szans na skok do np 12.5-14"
- board text removed: "Jak jest miejsce, to spokojnie rób szersze ścieżki na zasilanie. W razie czego puści więcej prądu, nie będzie brzydkich spadków itp."
- board text removed: "Poddtrzymuję, dodatkowy kondek tutaj nie zaszkodzi"
- board text removed: "Te przelotki tu nic nie wniosą jbc. Ścieżki są i tak za daleko od siebie"
